Commit message: update construction vr

File: gerri/robot/examples/construction_vr/m1509_urdf/m1509.urdf (robot description, URDF)
Before this commit: robot m1509, 8 links, 7 joints
Links:
- link base_link: geometry collision mesh filename=m1509_collision/MF1509_0_0.dae scale=0.001 0.001 0.001; visual mesh filename=m1509_blue/MF1509_0_0.dae scale=0.001 0.001 0.001
- link link_1: geometry collision mesh filename=m1509_collision/MF1509_1_0.dae scale=0.001 0.001 0.001; visual mesh filename=m1509_blue/MF1509_1_0.dae scale=0.001 0.001 0.001
- link link_2: geometry collision mesh filename=m1509_collision/MF1509_2_0.dae scale=0.001 0.001 0.001; collision mesh filename=m1509_collision/MF1509_2_1.dae scale=0.001 0.001 0.001
- link link_3: geometry collision mesh filename=m1509_collision/MF1509_3_0.dae scale=0.001 0.001 0.001; visual mesh filename=m1509_blue/MF1509_3_0.dae scale=0.001 0.001 0.001
- link link_4: geometry collision mesh filename=m1509_collision/MF1509_4_0.dae scale=0.001 0.001 0.001; collision mesh filename=m1509_collision/MF1509_4_1.dae scale=0.001 0.001 0.001
- link link_5: geometry collision mesh filename=m1509_collision/MF1509_5_0.dae scale=0.001 0.001 0.001; visual mesh filename=m1509_blue/MF1509_5_0.dae scale=0.001 0.001 0.001
- link link_6: geometry collision mesh filename=m1509_collision/MF1509_6_0.dae scale=0.001 0.001 0.001; visual mesh filename=m1509_blue/MF1509_6_0.dae scale=0.001 0.001 0.001
